Commit message: trying this on linux

File: body.urdf (robot description, URDF)
Before this commit: robot robot, 2 links, 1 joints
Links:
- removed link Link0
- removed link Link1
- added link BackLeg, mass 1; collision box size=1 1 1; visual box size=1 1 1
- added link FrontLeg, mass 1; collision box size=1 1 1; visual box size=1 1 1
- added link Torso, mass 1; collision box size=1 1 1; visual box size=1 1 1
Joints:
- removed joint Link0_Link1
- added joint Torso_BackLeg: type revolute, parent Torso, child BackLeg, origin xyz=-0.5 0 1.0 rpy=0 0 0, axis 0 1 0, limit lower=-3.14159 upper=3.14159 effort=0.0 velocity=0.0
- added joint Torso_FrontLeg: type revolute, parent Torso, child FrontLeg, origin xyz=0.5 0 1.0 rpy=0 0 0, axis 0 1 0, limit lower=-3.14159 upper=3.14159 effort=0.0 velocity=0.0

Commit message: quadruped submit

File: body.urdf (robot description, URDF)
Before this commit: robot robot, 3 links, 2 joints
Links:
- added link LeftLeg, mass 1; collision box size=1 0.2 0.2; visual box size=1 0.2 0.2
- added link LowerBack, mass 1; collision box size=0.2 0.2 1; visual box size=0.2 0.2 1
- added link LowerFront, mass 1; collision box size=0.2 0.2 1; visual box size=0.2 0.2 1
- added link LowerLeft, mass 1; collision box size=0.2 0.2 1; visual box size=0.2 0.2 1
- added link LowerRight, mass 1; collision box size=0.2 0.2 1; visual box size=0.2 0.2 1
- added link RightLeg, mass 1; collision box size=1 0.2 0.2; visual box size=1 0.2 0.2
- link BackLeg: geometry collision box size=0.2 1 0.2; visual box size=0.2 1 0.2
- link FrontLeg: geometry collision box size=0.2 1 0.2; visual box size=0.2 1 0.2
Joints:
- added joint BackLeg_LowerBack: type revolute, parent BackLeg, child LowerBack, origin xyz=0 -1 0 rpy=0 0 0, axis 1 0 0, limit lower=-3.14159 upper=3.14159 effort=0.0 velocity=0.0
- added joint FrontLeg_LowerFront: type revolute, parent FrontLeg, child LowerFront, origin xyz=0 1 0 rpy=0 0 0, axis 1 0 0, limit lower=-3.14159 upper=3.14159 effort=0.0 velocity=0.0
- added joint LeftLeg_LowerLeft: type revolute, parent LeftLeg, child LowerLeft, origin xyz=-1 0 0 rpy=0 0 0, axis 0 1 0, limit lower=-3.14159 upper=3.14159 effort=0.0 velocity=0.0
- added joint RightLeg_LowerRight: type revolute, parent RightLeg, child LowerRight, origin xyz=1 0 0 rpy=0 0 0, axis 0 1 0, limit lower=-3.14159 upper=3.14159 effort=0.0 velocity=0.0
- added joint Torso_LeftLeg: type revolute, parent Torso, child LeftLeg, origin xyz=-0.5 0 1 rpy=0 0 0, axis 0 1 0, limit lower=-3.14159 upper=3.14159 effort=0.0 velocity=0.0
- added joint Torso_RightLeg: type revolute, parent Torso, child RightLeg, origin xyz=0.5 0 1 rpy=0 0 0, axis 0 1 0, limit lower=-3.14159 upper=3.14159 effort=0.0 velocity=0.0
- joint Torso_BackLeg: axis 0 1 0 -> 1 0 0; origin xyz=-0.5 0 1.0 rpy=0 0 0 -> xyz=0 -0.5 1 rpy=0 0 0
- joint Torso_FrontLeg: axis 0 1 0 -> 1 0 0; origin xyz=0.5 0 1.0 rpy=0 0 0 -> xyz=0 0.5 1 rpy=0 0 0

Commit message: new body

File: body.urdf (robot description, URDF)
Before this commit: robot robot, 9 links, 8 joints
Links:
- removed link BackLeg
- removed link FrontLeg
- removed link LeftLeg
- removed link LowerBack
- removed link LowerFront
- removed link LowerLeft
- removed link LowerRight
- removed link RightLeg
- added link BackLeftLeg, mass 1; collision box size=0.2 0.2 1; visual box size=0.2 0.2 1
- added link BackLeftLower, mass 1; collision box size=0.2 0.2 1; visual box size=0.2 0.2 1
- added link BackRightLeg, mass 1; collision box size=0.2 0.2 1; visual box size=0.2 0.2 1
- added link BackRightLower, mass 1; collision box size=0.2 0.2 1; visual box size=0.2 0.2 1
- added link FrontLeftLeg, mass 1; collision box size=0.2 0.2 1; visual box size=0.2 0.2 1
- added link FrontLeftLower, mass 1; collision box size=0.2 0.2 1; visual box size=0.2 0.2 1
- added link FrontRightLeg, mass 1; collision box size=0.2 0.2 1; visual box size=0.2 0.2 1
- added link FrontRightLower, mass 1; collision box size=0.2 0.2 1; visual box size=0.2 0.2 1
- link Torso: geometry collision box size=3 1 1; visual box size=3 1 1
Joints:
- removed joint BackLeg_LowerBack
- removed joint FrontLeg_LowerFront
- removed joint LeftLeg_LowerLeft
- removed joint RightLeg_LowerRight
- removed joint Torso_BackLeg
- removed joint Torso_FrontLeg
- removed joint Torso_LeftLeg
- removed joint Torso_RightLeg
- added joint BackLeftLeg_BackLeftLower: type revolute, parent BackLeftLeg, child BackLeftLower, origin xyz=0 0 -1 rpy=0 0 0, axis 0 1 0, limit lower=-3.14159 upper=3.14159 effort=0.0 velocity=0.0
- added joint BackRightLeg_BackRightLower: type revolute, parent BackRightLeg, child BackRightLower, origin xyz=0 0 -1 rpy=0 0 0, axis 0 1 0, limit lower=-3.14159 upper=3.14159 effort=0.0 velocity=0.0
- added joint FrontLeftLeg_FrontLeftLower: type revolute, parent FrontLeftLeg, child FrontLeftLower, origin xyz=0 0 -1 rpy=0 0 0, axis 0 1 0, limit lower=-3.14159 upper=3.14159 effort=0.0 velocity=0.0
- added joint FrontRightLeg_FrontRightLower: type revolute, parent FrontRightLeg, child FrontRightLower, origin xyz=0 0 -1 rpy=0 0 0, axis 0 1 0, limit lower=-3.14159 upper=3.14159 effort=0.0 velocity=0.0
- added joint Torso_BackLeftLeg: type revolute, parent Torso, child BackLeftLeg, origin xyz=1.5 -0.5 2.0 rpy=0 0 0, axis 0 1 0, limit lower=-3.14159 upper=3.14159 effort=0.0 velocity=0.0
- added joint Torso_BackRightLeg: type revolute, parent Torso, child BackRightLeg, origin xyz=1.5 0.5 2.0 rpy=0 0 0, axis 0 1 0, limit lower=-3.14159 upper=3.14159 effort=0.0 velocity=0.0
- added joint Torso_FrontLeftLeg: type revolute, parent Torso, child FrontLeftLeg, origin xyz=-1.5 -0.5 2.0 rpy=0 0 0, axis 0 1 0, limit lower=-3.14159 upper=3.14159 effort=0.0 velocity=0.0
- added joint Torso_FrontRightLeg: type revolute, parent Torso, child FrontRightLeg, origin xyz=-1.5 0.5 2.0 rpy=0 0 0, axis 0 1 0, limit lower=-3.14159 upper=3.14159 effort=0.0 velocity=0.0

Commit message: changed fitness function to maximize time aloft

File: body.urdf (robot description, URDF)
Before this commit: robot robot, 9 links, 8 joints
Links:
- link Torso: geometry collision box size=3 2 0.5; visual box size=3 2 0.5
Joints:
- joint Torso_BackLeftLeg: origin xyz=1.5 -0.5 2.0 rpy=0 0 0 -> xyz=1.5 -1.0 2.25 rpy=0 0 0
- joint Torso_BackRightLeg: origin xyz=1.5 0.5 2.0 rpy=0 0 0 -> xyz=1.5 1.0 2.25 rpy=0 0 0
- joint Torso_FrontLeftLeg: origin xyz=-1.5 -0.5 2.0 rpy=0 0 0 -> xyz=-1.5 -1.0 2.25 rpy=0 0 0
- joint Torso_FrontRightLeg: origin xyz=-1.5 0.5 2.0 rpy=0 0 0 -> xyz=-1.5 1.0 2.25 rpy=0 0 0
